File: keyboard.kicad_sch (KiCad schematic)
At the start: 172 parts

Commit message: pasted esp32
Parts:
- added U1: ESP32-S3-WROOM-1, RF_Module:ESP32-S3-WROOM-1, symbol RF_Module:ESP32-S3-WROOM-1
Connections:
- new net: U1.1 (GND), U1.40 (GND), U1.41 (GND)
Other:
- note added: "if we want just a chip then we need to either buy flash on package or design own"
Changed lines of the file:
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@@
 		)
 	)
+	(text "if we want just a chip then we need to either buy flash on package or design own\n"
+		(exclude_from_sim no)
+		(at 402.336 217.932 0)
+		(effects
+			(font
+				(size 1.27 1.27)
+			)
+		)
+	)
 	(junction
 		(at 135.89 35.56)
@@
 					(unit 1)
 				)
+			)
+		)
+	)
+	(symbol
+		(lib_id "RF_Module:ESP32-S3-WROOM-1")
+		(at 422.91 137.16 0)
+		(unit 1)
+		(body_style 1)
+		(exclude_from_sim no)
+		(in_bom yes)
+		(on_board yes)
+		(in_pos_files yes)
+		(dnp no)
+		(fields_autoplaced yes)
+		(property "Reference" "U1"
+			(at 425.0533 106.68 0)
+			(show_name no)
+			(do_not_autoplace no)
+			(effects
+				(font
+					(size 1.27 1.27)
+				)
+				(justify left)
+			)
+		)
+		(property "Value" "ESP32-S3-WROOM-1"
+			(at 425.0533 109.22 0)
+			(show_name no)
+			(do_not_autoplace no)
+			(effects
+				(font
+					(size 1.27 1.27)
+				)
+				(justify left)
+			)
+		)
+		(property "Footprint" "RF_Module:ESP32-S3-WROOM-1"
+			(at 422.91 134.62 0)
+			(hide yes)
+			(show_name no)
+			(do_not_autoplace no)
+			(effects
+				(font
+					(size 1.27 1.27)
+				)
+			)
+		)
+		(property "Datasheet" "https://www.espressif.com/sites/default/files/documentation/esp32-s3-wroom-1_wroom-1u_datasheet_en.pdf"
+			(at 422.91 137.16 0)
+			(hide yes)
+			(show_name no)
+			(do_not_autoplace no)
+			(effects
+				(font
+					(size 1.27 1.27)
+				)
+			)
+		)
+		(property "Description" "RF Module, ESP32-S3 SoC, Wi-Fi 802.11b/g/n, Bluetooth, BLE, 32-bit, 3.3V, onboard antenna, SMD"
+			(at 422.91 137.16 0)
+			(hide yes)
+			(show_name no)
+			(do_not_autoplace no)
+			(effects
+				(font
+					(size 1.27 1.27)
+				)
+			)
+		)
+		(pin "10"
+		)
+		(pin "14"
+		)
+		(pin "9"
+		)
+		(pin "17"
+		)
+		(pin "19"
+		)
+		(pin "6"
+		)
+		(pin "13"
+		)
+		(pin "4"
+		)
+		(pin "3"
+		)
+		(pin "7"
+		)
+		(pin "8"
+		)
+		(pin "2"
+		)
+		(pin "5"
+		)
+		(pin "11"
+		)
+		(pin "1"
+		)
+		(pin "12"
+		)
+		(pin "15"
+		)
+		(pin "16"
+		)
+		(pin "18"
+		)
+		(pin "36"
+		)
+		(pin "38"
+		)
+		(pin "30"
+		)
+		(pin "35"
+		)
+		(pin "29"
+		)
+		(pin "31"
+		)
+		(pin "40"
+		)
+		(pin "32"
+		)
+		(pin "27"
+		)
+		(pin "22"
+		)
+		(pin "28"
+		)
+		(pin "24"
+		)
+		(pin "23"
+		)
+		(pin "33"
+		)
+		(pin "39"
+		)
+		(pin "20"
+		)
+		(pin "41"
+		)
+		(pin "25"
+		)
+		(pin "26"
+		)
+		(pin "34"
+		)
+		(pin "21"
+		)
+		(pin "37"
+		)
+		(instances
+			(project "keyboard"
+				(path "/c605602d-1549-47d7-8838-386321d100e9"
+					(reference "U1")
+					(unit 1)
+				)
