File: keyboard.kicad_pcb (KiCad board)
At the start: 2 copper layers, 394.5 x 131.8 mm, 176 parts, among them SW1 RotaryEncoder, U1 ESP32-DevKitC

Commit message: added led and encoders
Parts:
- removed U1: ESP32-DevKitC, PCM_Espressif:ESP32-DevKitC
